Commit message: feat: stage 2 done

File: digital-twin-and-teleoperation/public/assets/industrial-5axis-arm.urdf (robot description, URDF)
Before this commit: robot industrial_5axis_arm, 12 links, 11 joints
Links:
- added link finger_left; visual box size=0.018 0.03 0.09
- added link finger_right; visual box size=0.018 0.03 0.09
- link tool0: geometry visual cylinder length=0.04 radius=0.045
Joints:
- added joint finger_left_joint: type prismatic, parent tool0, child finger_left, origin xyz=0 0 0.04 rpy=0 0 0, axis 0 -1 0, limit lower=0 upper=0.03 effort=20 velocity=0.1
- added joint finger_right_joint: type prismatic, parent tool0, child finger_right, origin xyz=0 0 0.04 rpy=0 0 0, axis 0 1 0, limit lower=0 upper=0.03 effort=20 velocity=0.1
- joint base_to_joint1_housing: origin xyz=0 0 0.15 rpy=0 0 0 -> xyz=0 0 0.075 rpy=0 0 0
- joint joint1: origin xyz=0 0 0 rpy=0 0 0 -> xyz=0 0 0.1 rpy=0 0 0

Commit message: update: urdf

File: digital-twin-and-teleoperation/public/assets/industrial-5axis-arm.urdf (robot description, URDF)
Before this commit: robot industrial_5axis_arm, 14 links, 13 joints
Links:
- removed link joint1_housing
- removed link joint2_housing
- removed link joint3_housing
- removed link joint4_housing
- removed link joint5_housing
- removed link link1
- removed link link2
- removed link link3
- removed link link4
- removed link link5
- removed link tool0
- added link gripper_base; visual box size=0.02 0.08 0.03
- added link link_1; visual cylinder length=0.2 radius=0.07
- added link link_2; visual cylinder length=0.02 radius=0.085; visual cylinder length=0.08 radius=0.075
- added link link_3; visual cylinder length=0.01 radius=0.07; visual cylinder length=0.08 radius=0.065
- added link link_4; visual cylinder length=0.05 radius=0.04; visual cylinder length=0.05 radius=0.05
- added link link_5; visual cylinder length=0.03 radius=0.035; visual sphere radius=0.038
- link base_link: geometry visual box size=0.25 0.25 0.06
- link finger_left: geometry visual box size=0.01 0.003 0.014; visual box size=0.04 0.008 0.018
- link finger_right: geometry visual box size=0.01 0.003 0.014; visual box size=0.04 0.008 0.018
Joints:
- removed joint base_to_joint1_housing
- removed joint finger_left_joint
- removed joint finger_right_joint
- removed joint joint1
- removed joint joint2
- removed joint joint3
- removed joint joint4
- removed joint joint5
- removed joint link1_to_joint2_housing
- removed joint link2_to_joint3_housing
- removed joint link3_to_joint4_housing
- removed joint link4_to_joint5_housing
- removed joint link5_to_tool0
- added joint joint_1: type revolute, parent base_link, child link_1, origin xyz=0 0 0.06 rpy=0 0 0, axis 0 0 1, limit lower=-3.14 upper=3.14 effort=100 velocity=2
- added joint joint_2: type revolute, parent link_1, child link_2, origin xyz=0 0 0.2 rpy=0 0 0, axis 0 1 0, limit lower=-1.57 upper=1.57 effort=100 velocity=2
- added joint joint_3: type revolute, parent link_2, child link_3, origin xyz=0 0 0.4 rpy=0 0 0, axis 0 1 0, limit lower=-2.0 upper=2.0 effort=80 velocity=2.5
- added joint joint_4: type revolute, parent link_3, child link_4, origin xyz=0.35 0 0 rpy=0 0 0, axis 1 0 0, limit lower=-3.14 upper=3.14 effort=50 velocity=3
- added joint joint_5: type revolute, parent link_4, child link_5, origin xyz=0.1 0 0 rpy=0 0 0, axis 0 1 0, limit lower=-1.57 upper=1.57 effort=30 velocity=3
- added joint joint_finger_left: type prismatic, parent gripper_base, child finger_left, origin xyz=0.03 -0.025 0 rpy=0 0 0, axis 0 1 0, limit lower=0 upper=0.02 effort=20 velocity=0.1
- added joint joint_finger_right: type prismatic, parent gripper_base, child finger_right, origin xyz=0.03 0.025 0 rpy=0 0 0, axis 0 -1 0, limit lower=0 upper=0.02 effort=20 velocity=0.1
- added joint joint_gripper_base: type fixed, parent link_5, child gripper_base, origin xyz=0.03 0 0 rpy=0 0 0
